Commit message: adjusted mycobot files for Ros2 Humble

File: mycobot_description/urdf/sensors/intel_rgbd_cam_d435.urdf.xacro (robot description, xacro)
@@ -29,5 +29,5 @@
       </visual>
       <visual name="base">
-        <origin xyz="0 0 0" rpy="0 0 0" />
+        <origin xyz="0 0 0.03" rpy="0 0 0" />
         <material name="LightGrey">
           <color rgba="0.7 0.7 0.7 1.0"/>
@@ -40,9 +40,9 @@
         <origin xyz="0 0 0.25" rpy="0 0 0" />
         <geometry>
-          <cylinder radius="0.005" length="0.6"/>
+          <cylinder radius="0.005" length="0.5"/>
         </geometry>
       </collision>
       <collision name="base">
-        <origin xyz="0 0 0.0" rpy="0 0 0" />
+        <origin xyz="0 0 0.03" rpy="0 0 0" />
         <geometry>
           <box size="0.15 0.10 0.06" />
