Commit message: Bring the eye-to-hand calibration up on real hardware
Runs the same pipeline on the physical myCobot 280 and in simulation, and
records what the hardware taught us about the target and the sweep.

Camera over the network. The D435 sits on a JetBot on another subnet running
Eloquent, so the two ROS graphs cannot be joined. jetbot_frame_server.py is a
plain TCP frame pusher with no ROS dependency; jetbot_camera_bridge republishes
on the simulation's own topic names so the detector, collector and solver run
unmodified. hardware_overrides.yaml carries only the values that differ and
inherits the rest, so sim and hardware cannot drift apart silently.

The 38 mm target is the central limitation. A planar marker's pose has two
solutions separated only by foreshortening, and past ~0.29 m
SOLVEPNP_IPPE_SQUARE flips between them: 174.6 deg of rotation spread with the
arm completely stationary at 0.32 m, against 1.49 deg at 0.222 m. The cap must
come from the ROTATION, not the position -- translation is still sub-millimetre
at 0.287 m where rotation has already collapsed, so a cap chosen from position
data alone still let every pose fail. Tilt does not help; range is the whole
story. Hence max_marker_distance, defaulting to 0 (off) because simulation's
clean corners resolve the ambiguity at far smaller pixel counts.

settle_time goes to 3.5 s on hardware. Classifying one sweep's 77 rejected
poses by how they failed put 67 in the "both translation and rotation moved"
bucket, which is a coasting arm, against 10 rotation-only, which is ambiguity.
Settling was 87% of the loss. That plus correcting nominal_camera_position took
captures from 5/146 to 40/121.

Ctrl-C now keeps the samples already collected. Until this, an interrupt threw
away the whole sweep: write_dataset ran only after the loop and main() caught
KeyboardInterrupt just to log it.

The simulated camera moves to the pose measured on the physical rig, so both
see the same geometry from 0.5235 m. Fifteen places carry that pose and all had
to move together; the launch files declare their own defaults and pass them to
xacro, so editing only the xacro changes nothing.

RViz configs are derived from one RViz itself wrote. An Image display lives in
a Qt dock that is positioned only by the QMainWindow State blob, so a
hand-written config loads clean, subscribes, receives every frame, and draws
nothing.

Results in results/ with a top-level README covering both paths. Three
independent 40-sample hardware sweeps agree on the camera to 14.3 mm and
5.9 deg, which is the honest uncertainty for a 38 mm target on this rig.

Known and unfixed: handeye_solver and pose_collector both hardcode
camera_head_depth_optical_frame while the hardware detector stamps the colour
frame, and present_target_node uses is_reachable's (ok, message) tuple as a
bare truth value so its reachability gate never fires.

Co-Authored-By: Claude Opus 5 <noreply@anthropic.com>
Claude-Session: https://claude.ai/code/session_016tpJeR2w2Qxa27VWPcvbdF

File: mycobot_description/urdf/sensors/intel_rgbd_cam_d435.urdf.xacro (robot description, xacro)
@@ -94,6 +94,6 @@
     that does not detect. Trust a detection over the coverage score.
   -->
-  <xacro:arg name="camera_tilt_deg" default="24.45"/>
-  <xacro:arg name="camera_pan_deg" default="119.14"/>
+  <xacro:arg name="camera_tilt_deg" default="23.97"/>
+  <xacro:arg name="camera_pan_deg" default="162.13"/>
   <!--
     Where the stand is, in base_link. Exposed so the camera can be moved
@@ -147,7 +147,20 @@
   <xacro:arg name="camera_offset_y" default="-0.025"/>
   <xacro:arg name="camera_offset_z" default="0.0"/>
-  <xacro:arg name="camera_stand_x" default="0.287"/>
-  <xacro:arg name="camera_stand_y" default="0.160"/>
-  <xacro:arg name="camera_stand_z" default="0.45"/>
+  <xacro:arg name="camera_stand_x" default="0.1666"/>
+  <xacro:arg name="camera_stand_y" default="0.2575"/>
+  <xacro:arg name="camera_stand_z" default="0.4330"/>
+  <!-- How far BELOW base_link the stand's foot reaches, in metres.
+       The stand hangs off base_link, so its foot sits at base_link's height
+       and rests on the table only while base_link is exactly level with the
+       table top. It is not, so without this the stand floats or sinks.
+       Keep it equal to (spawn z - 0.425). NEGATIVE is legal and currently
+       correct: at spawn z 0.410 the foot must reach UP 0.015 to meet the
+       table. The arithmetic works either way: the pole runs from minus drop
+       up to camera_stand_z, so it spans 0.015 to 0.4330 here.
+       This extends the foot downwards ONLY. The camera stays at
+       camera_stand_z above base_link, which is the pose measured on the
+       physical rig and the only geometry the calibration sees, so changing
+       this is purely cosmetic. -->
+  <xacro:arg name="camera_stand_drop" default="0.035"/>
   <xacro:if value="${'true' == '$(arg use_camera)' and 'true' == '$(arg use_gazebo)'}">
     <xacro:property name="M_PI" value="3.1415926535897931" />
@@ -167,14 +180,14 @@
       </inertial>
       <visual name="holder">
-        <origin xyz="0 0 ${$(arg camera_stand_z)/2}" rpy="0 0 0" />
+        <origin xyz="0 0 ${($(arg camera_stand_z) - $(arg camera_stand_drop))/2}" rpy="0 0 0" />
         <material name="LightGrey">
           <color rgba="0.7 0.7 0.7 1.0"/>
         </material>
         <geometry>
-          <cylinder radius="0.005" length="$(arg camera_stand_z)"/>
+          <cylinder radius="0.005" length="${$(arg camera_stand_z) + $(arg camera_stand_drop)}"/>
         </geometry>
       </visual>
       <visual name="base">
-        <origin xyz="0 0 0.03" rpy="0 0 0" />
+        <origin xyz="0 0 ${0.03 - $(arg camera_stand_drop)}" rpy="0 0 0" />
         <material name="LightGrey">
           <color rgba="0.7 0.7 0.7 1.0"/>
@@ -185,11 +198,11 @@
       </visual>
       <collision name="holder">
-        <origin xyz="0 0 ${$(arg camera_stand_z)/2}" rpy="0 0 0" />
-        <geometry>
-          <cylinder radius="0.005" length="$(arg camera_stand_z)"/>
+        <origin xyz="0 0 ${($(arg camera_stand_z) - $(arg camera_stand_drop))/2}" rpy="0 0 0" />
+        <geometry>
+          <cylinder radius="0.005" length="${$(arg camera_stand_z) + $(arg camera_stand_drop)}"/>
         </geometry>
       </collision>
       <collision name="base">
-        <origin xyz="0 0 0.03" rpy="0 0 0" />
+        <origin xyz="0 0 ${0.03 - $(arg camera_stand_drop)}" rpy="0 0 0" />
         <geometry>
           <box size="0.15 0.10 0.06" />
