Commit message: Gripper fixed, Tested AI agent Rosa for ROS2 topics

File: mycobot_description/urdf/control/mycobot_280_ros2_control.urdf.xacro (robot description, xacro)
@@ -58,4 +58,34 @@
                 <state_interface name="velocity"/>
             </joint>
+            <joint name="${prefix}gripper_base_to_${prefix}gripper_left2">
+                <param name="mimic">${prefix}gripper_controller</param>
+                <param name="multiplier">1.0</param>
+                <state_interface name="position"/>
+                <state_interface name="velocity"/>
+            </joint>
+            <joint name="${prefix}gripper_left3_to_${prefix}gripper_left1">
+                <param name="mimic">${prefix}gripper_controller</param>
+                <param name="multiplier">-1.0</param>
+                <state_interface name="position"/>
+                <state_interface name="velocity"/>
+            </joint>
+            <joint name="${prefix}gripper_base_to_${prefix}gripper_right3">
+                <param name="mimic">${prefix}gripper_controller</param>
+                <param name="multiplier">-1.0</param>
+                <state_interface name="position"/>
+                <state_interface name="velocity"/>
+            </joint>
+            <joint name="${prefix}gripper_base_to_${prefix}gripper_right2">
+                <param name="mimic">${prefix}gripper_controller</param>
+                <param name="multiplier">-1.0</param>
+                <state_interface name="position"/>
+                <state_interface name="velocity"/>
+            </joint>
+            <joint name="${prefix}gripper_right3_to_${prefix}gripper_right1">
+                <param name="mimic">${prefix}gripper_controller</param>
+                <param name="multiplier">1.0</param>
+                <state_interface name="position"/>
+                <state_interface name="velocity"/>
+            </joint>
         </ros2_control>
     </xacro:macro>

File: mycobot_description/urdf/mech/adaptive_gripper.urdf.xacro (robot description, xacro)
@@ -199,4 +199,30 @@
       </visual>
     </gazebo>
+    <!-- Dummy joints to satisfy MoveIt2 errors from gazebo_ros2_control appending _mimic -->
+    <link name="${prefix}dummy_mimic_link1"/>
+    <joint name="${prefix}gripper_base_to_${prefix}gripper_left2_mimic" type="fixed">
+      <parent link="${prefix}gripper_base"/>
+      <child link="${prefix}dummy_mimic_link1"/>
+    </joint>
+    <link name="${prefix}dummy_mimic_link2"/>
+    <joint name="${prefix}gripper_left3_to_${prefix}gripper_left1_mimic" type="fixed">
+      <parent link="${prefix}gripper_base"/>
+      <child link="${prefix}dummy_mimic_link2"/>
+    </joint>
+    <link name="${prefix}dummy_mimic_link3"/>
+    <joint name="${prefix}gripper_base_to_${prefix}gripper_right3_mimic" type="fixed">
+      <parent link="${prefix}gripper_base"/>
+      <child link="${prefix}dummy_mimic_link3"/>
+    </joint>
+    <link name="${prefix}dummy_mimic_link4"/>
+    <joint name="${prefix}gripper_base_to_${prefix}gripper_right2_mimic" type="fixed">
+      <parent link="${prefix}gripper_base"/>
+      <child link="${prefix}dummy_mimic_link4"/>
+    </joint>
+    <link name="${prefix}dummy_mimic_link5"/>
+    <joint name="${prefix}gripper_right3_to_${prefix}gripper_right1_mimic" type="fixed">
+      <parent link="${prefix}gripper_base"/>
+      <child link="${prefix}dummy_mimic_link5"/>
+    </joint>
   </xacro:macro>
 </robot>

File: mycobot_description/urdf/robots/mycobot_280.urdf.xacro (robot description, xacro)
@@ -10,5 +10,5 @@
     <xacro:arg name="use_camera" default="false"/>
     <xacro:arg name="use_gazebo" default="false"/>
-    <xacro:arg name="use_gripper" default="false"/>
+    <xacro:arg name="use_gripper" default="true"/>
     <xacro:if value="$(arg add_world)">
       <link name="world"/>
@@ -33,15 +33,10 @@
       <origin xyz="0 0 0" rpy="0 0 0"/>
     </xacro:mycobot_280_arm>
-    <xacro:if value="$(arg use_gripper)">
-        <xacro:property name="current_gripper" value="$(arg gripper_type)"/>
-        <xacro:if value="${current_gripper == 'adaptive_gripper'}">
-            <xacro:include filename="$(find mycobot_description)/urdf/mech/adaptive_gripper.urdf.xacro"/>
-            <xacro:adaptive_gripper
-                parent="$(arg flange_link)"
-                prefix="$(arg prefix)">
-                <origin xyz="0 0 0.034" rpy="1.579 0 0"/>
-            </xacro:adaptive_gripper>
-        </xacro:if>
-    </xacro:if>
+    <xacro:include filename="$(find mycobot_description)/urdf/mech/adaptive_gripper.urdf.xacro"/>
+    <xacro:adaptive_gripper
+        parent="$(arg flange_link)"
+        prefix="$(arg prefix)">
+        <origin xyz="0 0 0.034" rpy="1.579 0 0"/>
+    </xacro:adaptive_gripper>
     <xacro:include filename="$(find mycobot_description)/urdf/control/gazebo_sim_ros2_control.urdf.xacro" />
     <xacro:load_gazebo_sim_ros2_control_plugin
