Commit message: fix: update MoveIt start tolerance, hardware launch parameters, and SRDF group definitions

File: mycobot_description/urdf/control/mycobot_280_ros2_control.urdf.xacro (robot description, xacro)
@@ -1,5 +1,5 @@
 <?xml version="1.0" ?>
 <robot xmlns:xacro="http://wiki.ros.org/xacro">
-    <xacro:macro name="mycobot_ros2_control" params="prefix flange_link use_gazebo">
+    <xacro:macro name="mycobot_ros2_control" params="prefix flange_link use_gazebo use_gripper:=true">
         <ros2_control name="RobotSystem" type="system">
             <hardware>
@@ -7,4 +7,9 @@
                     <plugin>ign_ros2_control/IgnitionSystem</plugin>
                 </xacro:if>
+                <xacro:unless value="${use_gazebo}">
+                    <plugin>mycobot_hardware_interface/MyCobotSystemInterface</plugin>
+                    <param name="serial_port">/dev/ttyACM0</param>
+                    <param name="baud_rate">115200</param>
+                </xacro:unless>
             </hardware>
             <joint name="${prefix}link1_to_${prefix}link2">
@@ -50,42 +55,44 @@
                 <state_interface name="position"/>
             </joint>
-            <joint name="${prefix}gripper_controller">
-                <command_interface name="position">
-                    <param name="min">-0.7</param>
-                    <param name="max">0.15</param>
-                </command_interface>
-                <state_interface name="position"/>
-                <state_interface name="velocity"/>
-            </joint>
-            <joint name="${prefix}gripper_base_to_${prefix}gripper_left2">
-                <param name="mimic">${prefix}gripper_controller</param>
-                <param name="multiplier">1.0</param>
-                <state_interface name="position"/>
-                <state_interface name="velocity"/>
-            </joint>
-            <joint name="${prefix}gripper_left3_to_${prefix}gripper_left1">
-                <param name="mimic">${prefix}gripper_controller</param>
-                <param name="multiplier">-1.0</param>
-                <state_interface name="position"/>
-                <state_interface name="velocity"/>
-            </joint>
-            <joint name="${prefix}gripper_base_to_${prefix}gripper_right3">
-                <param name="mimic">${prefix}gripper_controller</param>
-                <param name="multiplier">-1.0</param>
-                <state_interface name="position"/>
-                <state_interface name="velocity"/>
-            </joint>
-            <joint name="${prefix}gripper_base_to_${prefix}gripper_right2">
-                <param name="mimic">${prefix}gripper_controller</param>
-                <param name="multiplier">-1.0</param>
-                <state_interface name="position"/>
-                <state_interface name="velocity"/>
-            </joint>
-            <joint name="${prefix}gripper_right3_to_${prefix}gripper_right1">
-                <param name="mimic">${prefix}gripper_controller</param>
-                <param name="multiplier">1.0</param>
-                <state_interface name="position"/>
-                <state_interface name="velocity"/>
-            </joint>
+            <xacro:if value="${use_gripper}">
+                <joint name="${prefix}gripper_controller">
+                    <command_interface name="position">
+                        <param name="min">-0.7</param>
+                        <param name="max">0.15</param>
+                    </command_interface>
+                    <state_interface name="position"/>
+                    <state_interface name="velocity"/>
+                </joint>
+                <joint name="${prefix}gripper_base_to_${prefix}gripper_left2">
+                    <param name="mimic">${prefix}gripper_controller</param>
+                    <param name="multiplier">1.0</param>
+                    <state_interface name="position"/>
+                    <state_interface name="velocity"/>
+                </joint>
+                <joint name="${prefix}gripper_left3_to_${prefix}gripper_left1">
+                    <param name="mimic">${prefix}gripper_controller</param>
+                    <param name="multiplier">-1.0</param>
+                    <state_interface name="position"/>
+                    <state_interface name="velocity"/>
+                </joint>
+                <joint name="${prefix}gripper_base_to_${prefix}gripper_right3">
+                    <param name="mimic">${prefix}gripper_controller</param>
+                    <param name="multiplier">-1.0</param>
+                    <state_interface name="position"/>
+                    <state_interface name="velocity"/>
+                </joint>
+                <joint name="${prefix}gripper_base_to_${prefix}gripper_right2">
+                    <param name="mimic">${prefix}gripper_controller</param>
+                    <param name="multiplier">-1.0</param>
+                    <state_interface name="position"/>
+                    <state_interface name="velocity"/>
+                </joint>
+                <joint name="${prefix}gripper_right3_to_${prefix}gripper_right1">
+                    <param name="mimic">${prefix}gripper_controller</param>
+                    <param name="multiplier">1.0</param>
+                    <state_interface name="position"/>
+                    <state_interface name="velocity"/>
+                </joint>
+            </xacro:if>
         </ros2_control>
     </xacro:macro>

File: mycobot_description/urdf/robots/mycobot_280.urdf.xacro (robot description, xacro)
@@ -47,5 +47,6 @@
       prefix="$(arg prefix)"
       flange_link="$(arg flange_link)"
-      use_gazebo="$(arg use_gazebo)"/>
+      use_gazebo="$(arg use_gazebo)"
+      use_gripper="$(arg use_gripper)"/>
     <xacro:include filename="$(find mycobot_description)/urdf/sensors/intel_rgbd_cam_d435.urdf.xacro"/>
 </robot>
