Commit message: fixed base texture and lightning

File: mycobot_description/urdf/mech/g_shape_base_v2_0.urdf.xacro (robot description, xacro)
@@ -24,10 +24,17 @@
             </collision>
         </link>
+        <!--
+          Unlike the arm links, this override is INTENTIONALLY kept enabled. base_link.dae is a
+          Rhino export with no texture image (and no PNG ships for it), so its own COLLADA
+          material is just a flat 0.98 off-white. A solid colour is the correct appearance here
+          anyway: the real G-shape base is plain anodised aluminium with no printed graphics.
+          Dark matte grey, deliberately darker than the light-grey textured arm links.
+        -->
         <gazebo reference="${prefix}${base_link}">
             <visual>
                 <material>
-                    <ambient>0.5 0.5 0.5 1</ambient>
-                    <diffuse>0.5 0.5 0.5 1</diffuse>
-                    <specular>0.5 0.5 0.5 1</specular>
+                    <ambient>0.12 0.12 0.12 1</ambient>
+                    <diffuse>0.22 0.22 0.22 1</diffuse>
+                    <specular>0.15 0.15 0.15 1</specular>
                 </material>
             </visual>

File: mycobot_description/urdf/mech/mycobot_280_arm.urdf.xacro (robot description, xacro)
@@ -40,5 +40,8 @@
           <mesh filename="file://$(find mycobot_description)/meshes/mycobot_280/visual/link1.dae"/>
         </geometry>
-        <origin xyz="0.0 0 0" rpy="0 0 ${-pi/2}"/>
+        <!-- No yaw: this mesh (Elephant Robotics export, like link2-7) is already authored
+             long-axis-in-Y and offset toward -Y, matching the collision box below. The old
+             Rhino mesh was long-axis-in-X and needed rpy="0 0 -pi/2". -->
+        <origin xyz="0.0 0 0" rpy="0 0 0"/>
       </visual>
       <collision>
